Commit message: Fix all issues
Signed-off-by: Rahul K.A <karahul209@gmail.com>

File: urdf/depth_camera.urdf.xacro (robot description, xacro)
@@ -11,5 +11,5 @@
         <origin xyz="0 0 0" rpy="0 0 0"/>
         <geometry>
-          <mesh filename="package://starling2-description/meshes/OakDLite.dae" scale="1 1 1"/>
+          <mesh filename="package://x500_description/meshes/camera/OakDLite.dae" scale="1 1 1"/>
         </geometry>
       </visual>

File: urdf/x500.urdf.xacro (robot description, xacro)
@@ -11,5 +11,5 @@
         <origin xyz="0 0 .025" rpy="0 0 3.141592654"/>
         <geometry>
-          <mesh filename="package://starling2-description/meshes/NXP-HGD-CF.dae" scale="1 1 1"/>
+          <mesh filename="package://x500_description/meshes/x500/NXP-HGD-CF.dae" scale="1 1 1"/>
         </geometry>
       </visual>
@@ -17,5 +17,5 @@
         <origin xyz="0.174 0.174 .032" rpy="0 0 -.45"/>
         <geometry>
-          <mesh filename="package://starling2-description/meshes/5010Base.dae" scale="1 1 1"/>
+          <mesh filename="package://x500_description/meshes/x500/5010Base.dae" scale="1 1 1"/>
         </geometry>
       </visual>
@@ -23,5 +23,5 @@
         <origin xyz="-0.174 0.174 .032" rpy="0 0 -.45"/>
         <geometry>
-          <mesh filename="package://starling2-description/meshes/5010Base.dae" scale="1 1 1"/>
+          <mesh filename="package://x500_description/meshes/x500/5010Base.dae" scale="1 1 1"/>
         </geometry>
       </visual>
@@ -29,5 +29,5 @@
         <origin xyz="0.174 -0.174 .032" rpy="0 0 -.45"/>
         <geometry>
-          <mesh filename="package://starling2-description/meshes/5010Base.dae" scale="1 1 1"/>
+          <mesh filename="package://x500_description/meshes/x500/5010Base.dae" scale="1 1 1"/>
         </geometry>
       </visual>
@@ -35,5 +35,5 @@
         <origin xyz="-0.174 -0.174 .032" rpy="0 0 -.45"/>
         <geometry>
-          <mesh filename="package://starling2-description/meshes/5010Base.dae" scale="1 1 1"/>
+          <mesh filename="package://x500_description/meshes/x500/5010Base.dae" scale="1 1 1"/>
         </geometry>
       </visual>
@@ -96,11 +96,11 @@
         <origin xyz="-0.022 -0.14638461538461536 -0.016" rpy="0 0 0"/>
         <geometry>
-          <mesh filename="package://starling2-description/meshes/1345_prop_ccw.stl" scale="0.8461538461538461 0.8461538461538461 0.8461538461538461"/>
-        </geometry>
-      </visual>
-      <visual>
-        <origin xyz="0 0 -.032" rpy="0 0 0"/>
-        <geometry>
-          <mesh filename="package://starling2-description/meshes/5010Bell.dae" scale="1 1 1"/>
+          <mesh filename="package://x500_description/meshes/x500/1345_prop_ccw.stl" scale="0.8461538461538461 0.8461538461538461 0.8461538461538461"/>
+        </geometry>
+      </visual>
+      <visual>
+        <origin xyz="0 0 -.032" rpy="0 0 0"/>
+        <geometry>
+          <mesh filename="package://x500_description/meshes/x500/5010Bell.dae" scale="1 1 1"/>
         </geometry>
       </visual>
@@ -127,11 +127,11 @@
         <origin xyz="-0.022 -0.14638461538461536 -0.016" rpy="0 0 0"/>
         <geometry>
-          <mesh filename="package://starling2-description/meshes/1345_prop_ccw.stl" scale="0.8461538461538461 0.8461538461538461 0.8461538461538461"/>
-        </geometry>
-      </visual>
-      <visual>
-        <origin xyz="0 0 -.032" rpy="0 0 0"/>
-        <geometry>
-          <mesh filename="package://starling2-description/meshes/5010Bell.dae" scale="1 1 1"/>
+          <mesh filename="package://x500_description/meshes/x500/1345_prop_ccw.stl" scale="0.8461538461538461 0.8461538461538461 0.8461538461538461"/>
+        </geometry>
+      </visual>
+      <visual>
+        <origin xyz="0 0 -.032" rpy="0 0 0"/>
+        <geometry>
+          <mesh filename="package://x500_description/meshes/x500/5010Bell.dae" scale="1 1 1"/>
         </geometry>
       </visual>
@@ -158,11 +158,11 @@
         <origin xyz="-0.022 -0.14638461538461536 -0.016" rpy="0 0 0"/>
         <geometry>
-          <mesh filename="package://starling2-description/meshes/1345_prop_cw.stl" scale="0.8461538461538461 0.8461538461538461 0.8461538461538461"/>
-        </geometry>
-      </visual>
-      <visual>
-        <origin xyz="0 0 -.032" rpy="0 0 0"/>
-        <geometry>
-          <mesh filename="package://starling2-description/meshes/5010Bell.dae" scale="1 1 1"/>
+          <mesh filename="package://x500_description/meshes/x500/1345_prop_cw.stl" scale="0.8461538461538461 0.8461538461538461 0.8461538461538461"/>
+        </geometry>
+      </visual>
+      <visual>
+        <origin xyz="0 0 -.032" rpy="0 0 0"/>
+        <geometry>
+          <mesh filename="package://x500_description/meshes/x500/5010Bell.dae" scale="1 1 1"/>
         </geometry>
       </visual>
@@ -189,11 +189,11 @@
         <origin xyz="-0.022 -0.14638461538461536 -0.016" rpy="0 0 0"/>
         <geometry>
-          <mesh filename="package://starling2-description/meshes/1345_prop_cw.stl" scale="0.8461538461538461 0.8461538461538461 0.8461538461538461"/>
-        </geometry>
-      </visual>
-      <visual>
-        <origin xyz="0 0 -.032" rpy="0 0 0"/>
-        <geometry>
-          <mesh filename="package://starling2-description/meshes/5010Bell.dae" scale="1 1 1"/>
+          <mesh filename="package://x500_description/meshes/x500/1345_prop_cw.stl" scale="0.8461538461538461 0.8461538461538461 0.8461538461538461"/>
+        </geometry>
+      </visual>
+      <visual>
+        <origin xyz="0 0 -.032" rpy="0 0 0"/>
+        <geometry>
+          <mesh filename="package://x500_description/meshes/x500/5010Bell.dae" scale="1 1 1"/>
         </geometry>
       </visual>

File: urdf/x500_depth.urdf.xacro (robot description, xacro)
@@ -2,7 +2,7 @@
 <robot name="x500_with_depth_camera" xmlns:xacro="http://ros.org/wiki/xacro">
   <!-- Include the x500 base macro -->
-  <xacro:include filename="$(find starling2-description)/urdf/x500.urdf.xacro"/>
+  <xacro:include filename="$(find x500_description)/urdf/x500.urdf.xacro"/>
   <!-- Include the depth camera macro -->
-  <xacro:include filename="$(find starling2-description)/urdf/depth_camera.urdf.xacro"/>
+  <xacro:include filename="$(find x500_description)/urdf/depth_camera.urdf.xacro"/>
   <!-- Instantiate the x500 base -->
   <xacro:x500_base name="x500">
@@ -11,5 +11,5 @@
   <!-- Attach the depth camera to the front of the drone -->
   <xacro:depth_camera name="front" parent="x500_base_link">
-    <origin xyz="0.1 0 0.05" rpy="0 0 0"/>
+    <origin xyz=".12 .03 .0" rpy="0 0 0"/>
   </xacro:depth_camera>
 </robot>

Commit message: Fix macro names
Signed-off-by: Rahul K.A <karahul209@gmail.com>

File: urdf/depth_camera.urdf.xacro (robot description, xacro)
@@ -2,5 +2,5 @@
 <robot name="OakD-Lite" xmlns:xacro="http://ros.org/wiki/xacro">
   <xacro:macro name="depth_camera" params="name parent *origin">
-    <link name="${name}_camera_link">
+    <link name="camera_link">
       <inertial>
         <mass value="0.061"/>
@@ -21,10 +21,10 @@
       </collision>
     </link>
-    <joint name="${name}_camera_joint" type="fixed">
+    <joint name="camera_joint" type="fixed">
       <parent link="${parent}"/>
-      <child link="${name}_camera_link"/>
+      <child link="camera_link"/>
       <xacro:insert_block name="origin"/>
     </joint>
-    <gazebo reference="${name}_camera_link">
+    <gazebo reference="camera_link">
       <sensor name="IMX214" type="camera">
         <pose>0.01233 -0.03 .01878 0 0 0</pose>

File: urdf/x500.urdf.xacro (robot description, xacro)
@@ -2,5 +2,5 @@
 <robot name="x500_base" xmlns:xacro="http://ros.org/wiki/xacro">
   <xacro:macro name="x500_base" params="name *origin">
-    <link name="${name}_base_link">
+    <link name="base_link">
       <inertial>
         <mass value="2.0"/>
@@ -87,5 +87,5 @@
       </collision>
     </link>
-    <link name="${name}_rotor_0">
+    <link name="rotor_0">
       <inertial>
         <mass value="0.016076923076923075"/>
@@ -112,11 +112,11 @@
       </collision>
     </link>
-    <joint name="${name}_rotor_0_joint" type="continuous">
-      <parent link="${name}_base_link"/>
-      <child link="${name}_rotor_0"/>
+    <joint name="rotor_0_joint" type="continuous">
+      <parent link="base_link"/>
+      <child link="rotor_0"/>
       <origin xyz="0.174 -0.174 0.06" rpy="0 0 0"/>
       <axis xyz="0 0 1"/>
     </joint>
-    <link name="${name}_rotor_1">
+    <link name="rotor_1">
       <inertial>
         <mass value="0.016076923076923075"/>
@@ -143,11 +143,11 @@
       </collision>
     </link>
-    <joint name="${name}_rotor_1_joint" type="continuous">
-      <parent link="${name}_base_link"/>
-      <child link="${name}_rotor_1"/>
+    <joint name="rotor_1_joint" type="continuous">
+      <parent link="base_link"/>
+      <child link="rotor_1"/>
       <origin xyz="-0.174 0.174 0.06" rpy="0 0 0"/>
       <axis xyz="0 0 1"/>
     </joint>
-    <link name="${name}_rotor_2">
+    <link name="rotor_2">
       <inertial>
         <mass value="0.016076923076923075"/>
@@ -174,11 +174,11 @@
       </collision>
     </link>
-    <joint name="${name}_rotor_2_joint" type="continuous">
-      <parent link="${name}_base_link"/>
-      <child link="${name}_rotor_2"/>
+    <joint name="rotor_2_joint" type="continuous">
+      <parent link="base_link"/>
+      <child link="rotor_2"/>
       <origin xyz="0.174 0.174 0.06" rpy="0 0 0"/>
       <axis xyz="0 0 1"/>
     </joint>
-    <link name="${name}_rotor_3">
+    <link name="rotor_3">
       <inertial>
         <mass value="0.016076923076923075"/>
@@ -205,11 +205,11 @@
       </collision>
     </link>
-    <joint name="${name}_rotor_3_joint" type="continuous">
-      <parent link="${name}_base_link"/>
-      <child link="${name}_rotor_3"/>
+    <joint name="rotor_3_joint" type="continuous">
+      <parent link="base_link"/>
+      <child link="rotor_3"/>
       <origin xyz="-0.174 -0.174 0.06" rpy="0 0 0"/>
       <axis xyz="0 0 1"/>
     </joint>
-    <gazebo reference="${name}_base_link">
+    <gazebo reference="base_link">
       <sensor name="air_pressure_sensor" type="air_pressure">
         <always_on>1</always_on>

File: urdf/x500_depth.urdf.xacro (robot description, xacro)
@@ -10,5 +10,5 @@
   </xacro:x500_base>
   <!-- Attach the depth camera to the front of the drone -->
-  <xacro:depth_camera name="front" parent="x500_base_link">
+  <xacro:depth_camera name="front" parent="base_link">
     <origin xyz=".12 .03 .0" rpy="0 0 0"/>
   </xacro:depth_camera>

Commit message: add camera lens frames
Signed-off-by: Rahul K.A <karahul209@gmail.com>

File: urdf/depth_camera.urdf.xacro (robot description, xacro)
@@ -25,4 +25,16 @@
       <child link="camera_link"/>
       <xacro:insert_block name="origin"/>
+    </joint>
+    <link name="rgb_link"/>
+    <link name="depth_link"/>
+    <joint name="rgb_joint" type="fixed">
+      <parent link="camera_link"/>
+      <child link="rgb_link"/>
+      <origin xyz="0.01233 -0.03 .01878 " rpy="0 0 0"/>
+    </joint>
+    <joint name="depth_joint" type="fixed">
+      <parent link="camera_link"/>
+      <child link="depth_link"/>
+      <origin xyz="0.01233 -0.03 .01878 " rpy="0 0 0"/>
     </joint>
     <gazebo reference="camera_link">

File: urdf/x500.urdf.xacro (robot description, xacro)
@@ -112,4 +112,11 @@
       </collision>
     </link>
+    <link name="odom_link">
+    </link>
+    <joint name="odom_joint" type="fixed">
+      <parent link="base_link"/>
+      <child link="odom_link"/>
+      <origin xyz="0 0 0" rpy="0 0 0"/>
+    </joint>
     <joint name="rotor_0_joint" type="continuous">
       <parent link="base_link"/>

Commit message: Update URDF to make camera REP compliant
Signed-off-by: Rahul K.A <karahul209@gmail.com>

File: urdf/depth_camera.urdf.xacro (robot description, xacro)
@@ -5,9 +5,9 @@
       <inertial>
         <mass value="0.061"/>
-        <origin xyz="0.00358 -0.03 .014" rpy="0 0 0"/>
+        <origin xyz="0.00358 -0.03 .014" rpy="0 0 0.0"/>
         <inertia ixx="0.0000460804" ixy="0" ixz="0" iyy="0.0000055421" iyz="0" izz="0.0000436519"/>
       </inertial>
       <visual>
-        <origin xyz="0 0 0" rpy="0 0 0"/>
+        <origin xyz="0 0 0" rpy="0.0 -1.5708 1.5708 "/>
         <geometry>
           <mesh filename="package://x500_description/meshes/camera/OakDLite.dae" scale="1 1 1"/>
@@ -15,5 +15,5 @@
       </visual>
       <collision>
-        <origin xyz="0.00358 -0.03 .014" rpy="0 0 0"/>
+        <origin xyz="0.00358 -0.03 .014" rpy="0.0 -1.5708 1.5708 "/>
         <geometry>
           <box size="0.0175 0.091 0.028"/>
@@ -25,16 +25,4 @@
       <child link="camera_link"/>
       <xacro:insert_block name="origin"/>
-    </joint>
-    <link name="rgb_link"/>
-    <link name="depth_link"/>
-    <joint name="rgb_joint" type="fixed">
-      <parent link="camera_link"/>
-      <child link="rgb_link"/>
-      <origin xyz="0.01233 -0.03 .01878 " rpy="0 0 0"/>
-    </joint>
-    <joint name="depth_joint" type="fixed">
-      <parent link="camera_link"/>
-      <child link="depth_link"/>
-      <origin xyz="0.01233 -0.03 .01878 " rpy="0 0 0"/>
     </joint>
     <gazebo reference="camera_link">

File: urdf/x500.urdf.xacro (robot description, xacro)
@@ -112,5 +112,5 @@
       </collision>
     </link>
-    <link name="odom_link">
+    <!-- <link name="odom_link">
     </link>
     <joint name="odom_joint" type="fixed">
@@ -118,5 +118,5 @@
       <child link="odom_link"/>
       <origin xyz="0 0 0" rpy="0 0 0"/>
-    </joint>
+    </joint> -->
     <joint name="rotor_0_joint" type="continuous">
       <parent link="base_link"/>

File: urdf/x500_depth.urdf.xacro (robot description, xacro)
@@ -11,5 +11,5 @@
   <!-- Attach the depth camera to the front of the drone -->
   <xacro:depth_camera name="front" parent="base_link">
-    <origin xyz=".12 .03 .0" rpy="0 0 0"/>
+    <origin xyz=".12 .03 .0" rpy="-1.5708 0.0 -1.5708"/>
   </xacro:depth_camera>
 </robot>
