Commit message: Add code
Signed-off-by: Rahul K.A <karahul209@gmail.com>

File: urdf/x500.urdf.xacro (robot description, xacro)
@@ -1,1740 +1,299 @@
-<?xml version="1.0" encoding="utf-8"?>
-<!-- This URDF was automatically created by SolidWorks to URDF Exporter! Originally created by Stephen Brawner (brawner@gmail.com)
-     Commit Version: 1.6.0-4-g7f85cfe  Build Version: 1.6.7995.38578
-     For more information, please see http://wiki.ros.org/sw_urdf_exporter -->
-<robot
-  name="starling2">
-  <link
-    name="base_link">
-    <inertial>
-      <origin
-        xyz="-0.000149374353086822 1.97259826530437E-05 0.0080312652423187"
-        rpy="0 0 0" />
-      <mass
-        value="0.0654572412672586" />
-      <inertia
-        ixx="0.0216666666666666"
-        ixy="1e-9"
-        ixz="1e-9"
-        iyy="0.02166666666666667"
-        iyz="1e-9"
-        izz="0.04000000000000001" />
-      </inertial>
-    <visual>
-      <origin
-        xyz="0 0 0"
-        rpy="0 0 0" />
-      <geometry>
-        <mesh
-          filename="file://$(find starling2_description)/meshes/base_link.STL" />
-      </geometry>
-      <material
-        name="">
-        <color
-          rgba="0.792156862745098 0.819607843137255 0.933333333333333 1" />
-      </material>
-    </visual>
-    <collision>
-      <origin
-        xyz="0 0 0"
-        rpy="0 0 0" />
-      <geometry>
-        <mesh
-          filename="file://$(find starling2_description)/meshes/base_link.STL" />
-      </geometry>
-    </collision>
-  </link>
-  <link
-    name="fl_foot_link">
-    <inertial>
-      <origin
-        xyz="-0.00264955845969433 -0.00523753503392298 -0.0233308820202257"
-        rpy="0 0 0" />
-      <mass
-        value="0.00507585684308429" />
-      <inertia
-        ixx="1e-9"
-        ixy="1e-9"
-        ixz="1e-9"
-        iyy="1e-9"
-        iyz="1e-9"
-        izz="1e-9" />
-    </inertial>
-    <visual>
-      <origin
-        xyz="0 0 0"
-        rpy="0 0 0" />
-      <geometry>
-        <mesh
-          filename="file://$(find starling2_description)/meshes/fl_foot_link.STL" />
-      </geometry>
-      <material
-        name="">
-        <color
-          rgba="0.792156862745098 0.819607843137255 0.933333333333333 1" />
-      </material>
-    </visual>
-    <!-- <collision>
-      <origin
-        xyz="0 0 0"
-        rpy="0 0 0" />
-      <geometry>
-        <mesh
-          filename="file://$(find starling2_description)/meshes/fl_foot_link.STL" />
-      </geometry>
-    </collision> -->
-  </link>
-  <joint
-    name="fl_foot_joint"
-    type="fixed">
-    <origin
-      xyz="0.0949999999999995 0.13 -0.00250000000000033"
-      rpy="0 0 0" />
-    <parent
-      link="base_link" />
-    <child
-      link="fl_foot_link" />
-    <axis
-      xyz="0 0 0" />
-  </joint>
-  <link
-    name="fl_motor_link">
-    <inertial>
-      <origin
-        xyz="7.13244564104487E-08 -2.12782971659164E-07 0.00923828850084918"
-        rpy="0 0 0" />
-      <mass
-        value="0.0197" />
-      <inertia
-        ixx="1e-9"
-        ixy="1e-9"
-        ixz="1e-9"
-        iyy="1e-9"
-        iyz="1e-9"
-        izz="1e-9" />
-    </inertial>
-    <visual>
-      <origin
-        xyz="0 0 0"
-        rpy="0 0 0" />
-      <geometry>
-        <mesh
-          filename="file://$(find starling2_description)/meshes/fl_motor_link.STL" />
-      </geometry>
-      <material
-        name="">
-        <color
-          rgba="0.792156862745098 0.819607843137255 0.933333333333333 1" />
-      </material>
-    </visual>
-    <collision>
-      <origin
-        xyz="0 0 0"
-        rpy="0 0 0" />
-        <geometry>
-            <cylinder radius="0.04" length="0.145"/>
-        </geometry>
-    </collision>
-  </link>
-  <joint
-    name="fl_motor_joint"
-    type="fixed">
-    <origin
-      xyz="0 0 0.00750000000000001"
-      rpy="0 0 0" />
-    <parent
-      link="fl_foot_link" />
-    <child
-      link="fl_motor_link" />
-    <axis
-      xyz="0 0 0" />
-  </joint>
-  <link
-    name="fl_rotor_link">
-    <inertial>
-      <origin
-        xyz="-3.32717593277965E-06 9.14219090292212E-07 0.0041505334731533"
-        rpy="0 0 0" />
-      <mass
-        value="0.00775420714403987" />
-      <inertia
-        ixx="3.8464910483993325e-07"
-        ixy="1e-9"
-        ixz="1e-9"
-        iyy="2.6115851691700804e-05"
-        iyz="1e-9"
-        izz="2.649858234714004e-05" />
-    </inertial>
-    <visual>
-      <origin
-        xyz="0 0 0"
-        rpy="0 0 0" />
-      <geometry>
-        <mesh
-          filename="file://$(find starling2_description)/meshes/fl_rotor_link.STL" />
-      </geometry>
-      <material
-        name="">
-        <color
-          rgba="0.792156862745098 0.819607843137255 0.933333333333333 1" />
-      </material>
-    </visual>
-    <!-- <collision>
-      <origin
-        xyz="0 0 0"
-        rpy="0 0 0" />
-      <geometry>
-        <mesh
-          filename="file://$(find starling2_description)/meshes/fl_rotor_link.STL" />
-      </geometry>
-    </collision> -->
-  </link>
-  <joint
-    name="fl_rotor_joint" type="revolute">
-    <origin
-      xyz="0 0 0.0145"
-      rpy="0 0 0" />
-    <parent
-      link="fl_motor_link" />
-    <child
-      link="fl_rotor_link" />
-    <axis
-      xyz="0 0 1" />
-    <limit lower="-1e+16" upper="1e+16" effort="1000" velocity="1000"/>
-  </joint>
-  <link
-    name="fl_rotor_nut_link">
-    <inertial>
-      <origin
-        xyz="-3.60788637160381E-08 6.08339327579088E-07 -0.00490418266988037"
-        rpy="0 0 0" />
-      <mass
-        value="0.000288814916439492" />
-      <inertia
-        ixx="1e-9"
-        ixy="1e-9"
-        ixz="1e-9"
-        iyy="1e-9"
-        iyz="1e-9"
-        izz="1e-9" />
-    </inertial>
-    <visual>
-      <origin
-        xyz="0 0 0"
-        rpy="0 0 0" />
-      <geometry>
-        <mesh
-          filename="file://$(find starling2_description)/meshes/fl_rotor_nut_link.STL" />
-      </geometry>
-      <material
-        name="">
-        <color
-          rgba="0.792156862745098 0.819607843137255 0.933333333333333 1" />
-      </material>
-    </visual>
-    <!-- <collision>
-      <origin
-        xyz="0 0 0"
-        rpy="0 0 0" />
-      <geometry>
-        <mesh
-          filename="file://$(find starling2_description)/meshes/fl_rotor_nut_link.STL" />
-      </geometry>
-    </collision> -->
-  </link>
-  <joint
-    name="fl_rotor_nut_joint"
-    type="fixed">
-    <origin
-      xyz="0 0 0.0296"
-      rpy="0 0 0" />
-    <parent
-      link="fl_motor_link" />
-    <child
-      link="fl_rotor_nut_link" />
-    <axis
-      xyz="0 0 0" />
-  </joint>
-  <link
-    name="fr_foot_link">
-    <inertial>
-      <origin
-        xyz="-0.00273643316219788 0.00542897719182416 -0.0242461349552204"
-        rpy="0 0 0" />
-      <mass
-        value="0.00490045874350842" />
-      <inertia
-        ixx="1e-9"
-        ixy="1e-9"
-        ixz="1e-9"
-        iyy="1e-9"
-        iyz="1e-9"
-        izz="1e-9" />
-    </inertial>
-    <visual>
-      <origin
-        xyz="0 0 0"
-        rpy="0 0 0" />
-      <geometry>
-        <mesh
-          filename="file://$(find starling2_description)/meshes/fr_foot_link.STL" />
-      </geometry>
-      <material
-        name="">
-        <color
-          rgba="0.792156862745098 0.819607843137255 0.933333333333333 1" />
-      </material>
-    </visual>
-    <!-- <collision>
-      <origin
-        xyz="0 0 0"
-        rpy="0 0 0" />
-      <geometry>
-        <mesh
-          filename="file://$(find starling2_description)/meshes/fr_foot_link.STL" />
-      </geometry>
-    </collision> -->
-  </link>
-  <joint
-    name="fr_foot_joint"
-    type="fixed">
-    <origin
-      xyz="0.095 -0.13 -0.0025"
-      rpy="0 0 0" />
-    <parent
-      link="base_link" />
-    <child
-      link="fr_foot_link" />
-    <axis
-      xyz="0 0 0" />
-  </joint>
-  <link
-    name="fr_motor_link">
-    <inertial>
-      <origin
-        xyz="2.13573664281652E-07 -6.89206864079583E-08 0.00923828850084922"
-        rpy="0 0 0" />
-      <mass
-        value="0.0197" />
-      <inertia
-        ixx="1e-9"
-        ixy="1e-9"
-        ixz="1e-9"
-        iyy="1e-9"
-        iyz="1e-9"
-        izz="1e-9" />
-    </inertial>
-    <visual>
-      <origin
-        xyz="0 0 0"
-        rpy="0 0 0" />
-      <geometry>
-        <mesh
-          filename="file://$(find starling2_description)/meshes/fr_motor_link.STL" />
-      </geometry>
-      <material
-        name="">
-        <color
-          rgba="0.792156862745098 0.819607843137255 0.933333333333333 1" />
-      </material>
-    </visual>
-    <collision>
-      <origin
-        xyz="0 0 0"
-        rpy="0 0 0" />
-        <geometry>
-            <cylinder radius="0.04" length="0.143"/>
-        </geometry>
-    </collision>
-  </link>
-  <joint
-    name="fr_motor_joint"
-    type="fixed">
-    <origin
-      xyz="0 0 0.00750000000000001"
-      rpy="0 0 0" />
-    <parent
-      link="fr_foot_link" />
-    <child
-      link="fr_motor_link" />
-    <axis
-      xyz="0 0 0" />
-  </joint>
-  <link
-    name="fr_rotor_link">
-    <inertial>
-      <origin
-        xyz="-1.34638191580383E-06 -7.75562652099993E-07 0.00414324904903203"
-        rpy="0 0 0" />
-      <mass
-        value="0.00811819594401099" />
-      <inertia
-        ixx="3.8464910483993325e-07"
-        ixy="1e-9"
-        ixz="1e-9"
-        iyy="2.6115851691700804e-05"
-        iyz="1e-9"
-        izz="2.649858234714004e-05" />
-    </inertial>
-    <visual>
-      <origin
-        xyz="0 0 0"
-        rpy="0 0 0" />
-      <geometry>
-        <mesh
-          filename="file://$(find starling2_description)/meshes/fr_rotor_link.STL" />
-      </geometry>
-      <material
-        name="">
-        <color
-          rgba="0.792156862745098 0.819607843137255 0.933333333333333 1" />
-      </material>
-    </visual>
-    <!-- <collision>
-      <origin
-        xyz="0 0 0"
-        rpy="0 0 0" />
-      <geometry>
-        <mesh
-          filename="file://$(find starling2_description)/meshes/fr_rotor_link.STL" />
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
Commit message: Increase x500 collision
Signed-off-by: Rahul K.A <karahul209@gmail.com>

File: urdf/x500.urdf.xacro (robot description, xacro)
@@ -59,5 +59,5 @@
         <origin xyz="0 0 .007" rpy="0 0 0"/>
         <geometry>
-          <box size="0.35355339059327373 0.35355339059327373 0.05"/>
+          <box size="1.0 1.0 1.0"/>
         </geometry>
       </collision>
